Commit message: added second lidar, updated world file, added template files

File: urdf/fella.gazebo.xacro (robot description, xacro)
@@ -2,4 +2,5 @@
 <robot name="fella" xmlns:xacro="http://ros.org/wiki/xacro">
   <xacro:arg name="laser_visual"  default="true" />
+  <xacro:arg name="secondary_laser_visual" default="true" />
   <xacro:arg name="camera_visual" default="true"/>
   <xacro:arg name="imu_visual"    default="false"/>
@@ -78,5 +79,5 @@
       filename="ignition-gazebo-velocity-control-system"
       name="ignition::gazebo::systems::VelocityControl">
-      <topic>fella/cmd_vel</topic>
+      <topic>/cmd_vel</topic>
     </plugin>
   </gazebo>
@@ -86,5 +87,5 @@
       filename="ignition-gazebo-odometry-publisher-system"
       name="ignition::gazebo::systems::OdometryPublisher">
-      <topic>fella/odometry</topic>
+      <topic>/odom</topic>
       <odom_publish_frequency>20</odom_publish_frequency>
       <odom_frame>odom</odom_frame>
@@ -112,4 +113,35 @@
       <visualize>$(arg laser_visual)</visualize>
       <topic>fella/scan</topic>
+      <update_rate>3</update_rate>
+      <gz_frame_id>base_scan</gz_frame_id>
+      <ray>
+        <scan>
+          <horizontal>
+            <samples>360</samples>
+            <resolution>1</resolution>
+            <min_angle>0.0</min_angle>
+            <max_angle>6.28319</max_angle>
+          </horizontal>
+        </scan>
+        <range>
+          <min>0.2</min>
+          <max>40</max>
+          <resolution>0.015</resolution>
+        </range>
+        <noise>
+          <type>gaussian</type>
+          <mean>0.0</mean>
+          <stddev>0.01</stddev>
+        </noise>
+      </ray>
+      <always_on>true</always_on>
+    </sensor>
+  </gazebo>
+    <gazebo reference="secondary_base_scan">
+    <material>Gazebo/FlatBlack</material>
+    <sensor type="gpu_lidar" name="secondary_lidar">
+      <pose relative_to='base_scan'>0 0 0 0 0 0</pose>
+      <visualize>$(arg secondary_laser_visual)</visualize>
+      <topic>fella/secondary_scan</topic>
       <update_rate>3</update_rate>
       <gz_frame_id>base_scan</gz_frame_id>

File: urdf/fella.urdf.xacro (robot description, xacro)
@@ -48,4 +48,9 @@
         <origin xyz="0 0 0.175" rpy="0 0 0"/>
     </joint>
+    <joint name="secondary_scan_joint" type="fixed">
+        <parent link = "base_link"/>
+        <child link="secondary_base_scan"/>
+        <origin xyz="0.12374 0.0 0.12374" rpy="0 0.785398 0"/>
+    </joint>
     <link name="base_scan">
         <visual>
@@ -55,4 +60,20 @@
             </geometry>
             <material name="dark"/>
+        </visual>
+        <inertial>
+            <mass value="0" />
+            <origin xyz="0 0 0" />
+            <inertia ixx="0.001" ixy="0.0" ixz="0.0"
+                    iyy="0.001" iyz="0.0"
+                    izz="0.001" />
+        </inertial>
+    </link>
+    <link name="secondary_base_scan">
+        <visual>
+            <origin xyz="0 0 0" rpy="0 0 0"/>
+            <geometry>
+                <cylinder length="0.04" radius="0.09"/>
+            </geometry>
+            <material name="green"/>
         </visual>
         <inertial>

Commit message: so confused

File: urdf/fella.gazebo.xacro (robot description, xacro)
@@ -11,5 +11,5 @@
       <visualize>$(arg imu_visual)</visualize>
       <update_rate>100</update_rate>
-      <topic>fella/imu</topic>
+      <topic>/fella/imu</topic>
       <gz_frame_id>imu_link</gz_frame_id>
       <imu>
@@ -98,5 +98,5 @@
       filename="ignition-gazebo-joint-state-publisher-system"
       name="ignition::gazebo::systems::JointStatePublisher">
-      <topic>fella/joint_states</topic>
+      <topic>/joint_states</topic>
     </plugin>
   </gazebo>
@@ -113,5 +113,5 @@
       <pose relative_to='base_scan'>0 0 0.2 0 0 0</pose>
       <visualize>$(arg laser_visual)</visualize>
-      <topic>fella/scan</topic>
+      <topic>/fella/scan</topic>
       <update_rate>3</update_rate>
       <gz_frame_id>base_scan</gz_frame_id>
@@ -144,5 +144,5 @@
       <pose relative_to='secondary_base_scan'>0 0 0 0 0 0</pose>
       <visualize>$(arg secondary_laser_visual)</visualize>
-      <topic>fella/secondary_scan</topic>
+      <topic>/fella/secondary_scan</topic>
       <update_rate>3</update_rate>
       <gz_frame_id>base_scan</gz_frame_id>
@@ -199,5 +199,5 @@
       <update_rate>3</update_rate> <!--10-->
       <visualize>$(arg camera_visual)</visualize>
-      <topic>fella/camera</topic>
+      <topic>/fella/camera</topic>
       <gz_frame_id>camera_link</gz_frame_id>
     </sensor>

File: urdf/fella.urdf.xacro (robot description, xacro)
@@ -17,5 +17,5 @@
         </visual>
         <collision name="base_link_collision">
-            <origin xyz="0 0 0.03282" rpy="1.5708 0 0"/>
+            <origin xyz="0.0 0 0.03282" rpy="1.5708 0 0"/>
             <geometry>
                 <cylinder radius="0.122" length="0.831"/>
@@ -23,5 +23,5 @@
         </collision>
         <inertial>
-            <origin xyz="0 0 0.03282" rpy="0 0 0"/>
+            <origin xyz="-0.1 0 0.03282" rpy="0 0 0"/>
             <mass value="20.0"/>
             <inertia
@@ -37,4 +37,7 @@
     <xacro:wheel wheel_id="left" y_pos="0.42" x_pos="0.0"/>
     <xacro:wheel wheel_id="right" y_pos="-0.42" x_pos="0.0"/>
+    <!-- more wheels but make them invisible -->
+    <!-- <xacro:wheel wheel_id="front" y_pos="0.0" x_pos="0.32"--> -->
+    <xacro:wheel wheel_id="back" y_pos="0.0" x_pos="-0.32"/>
     <joint name="imu_joint" type="fixed">
         <parent link="base_link"/>
