Commit message: multi robot code (broken)

File: urdf/fella.urdf.xacro (robot description, xacro)
@@ -4,9 +4,11 @@
     <xacro:include filename="$(find unomas)/urdf/fella.gazebo.xacro"/>
     <xacro:include filename="$(find unomas)/urdf/wheel.urdf.xacro"/>
+    <xacro:arg name="robot_name" default="fella"/>
+    <xacro:property name="robot_name" value="$(arg robot_name)"/>
     <xacro:property name="r200_cam_rgb_px" value="0.005"/>
     <xacro:property name="r200_cam_rgb_py" value="0.018"/>
     <xacro:property name="r200_cam_rgb_pz" value="0.013"/>
     <xacro:property name="r200_cam_depth_offset" value="0.01"/>
-    <link name="base_link">
+    <link name="${robot_name}_base_link">
         <visual>
             <origin xyz="0 0 0.03282" rpy="1.5708 0 3.1415"/>
@@ -16,5 +18,5 @@
             <material name="blue"/>
         </visual>
-        <collision name="base_link_collision">
+        <collision name="${robot_name}_base_link_collision">
             <origin xyz="0 0 0.03282" rpy="1.5708 0 0"/>
             <geometry>
@@ -37,16 +39,16 @@
     <xacro:wheel wheel_id="left" y_pos="0.42" x_pos="0.0"/>
     <xacro:wheel wheel_id="right" y_pos="-0.42" x_pos="0.0"/>
-    <joint name="imu_joint" type="fixed">
-        <parent link="base_link"/>
-        <child link="imu_link"/>
+    <joint name="${robot_name}_imu_joint" type="fixed">
+        <parent link="${robot_name}_base_link"/>
+        <child link="${robot_name}_imu_link"/>
         <origin xyz="0.0 0.0 0.0" rpy="0 0 0"/>
     </joint>
-    <link name="imu_link"/>
-    <joint name="scan_joint" type="fixed">
-        <parent link="base_link"/>
-        <child link="base_scan"/>
+    <link name="${robot_name}_imu_link"/>
+    <joint name="${robot_name}_scan_joint" type="fixed">
+        <parent link="${robot_name}_base_link"/>
+        <child link="${robot_name}_base_scan"/>
         <origin xyz="0 0 0.175" rpy="0 0 0"/>
     </joint>
-    <link name="base_scan">
+    <link name="${robot_name}_base_scan">
         <visual>
             <origin xyz="0 0 0" rpy="0 0 0"/>
@@ -64,10 +66,10 @@
         </inertial>
     </link>
-    <joint name="camera_joint" type="fixed">
+    <joint name="${robot_name}_camera_joint" type="fixed">
         <origin xyz="0.13 0.0 0.03282" rpy="0 0 0"/>
-        <parent link="base_link"/>
-        <child link="camera_link"/>
+        <parent link="${robot_name}_base_link"/>
+        <child link="${robot_name}_camera_link"/>
     </joint>
-    <link name="camera_link">
+    <link name="${robot_name}_camera_link">
         <visual>
             <origin xyz="0 0 0" rpy="0 0 0"/>
@@ -85,27 +87,27 @@
         </visual>
     </link>
-    <joint name="camera_rgb_joint" type="fixed">
+    <joint name="${robot_name}_camera_rgb_joint" type="fixed">
         <origin xyz="${r200_cam_rgb_px} ${r200_cam_rgb_py} ${r200_cam_rgb_pz}" rpy="0 0 0"/>
-        <parent link="camera_link"/>
-        <child link="camera_rgb_frame"/>
+        <parent link="${robot_name}_camera_link"/>
+        <child link="${robot_name}_camera_rgb_frame"/>
     </joint>
-    <link name="camera_rgb_frame"/>
-    <joint name="camera_rgb_optical_joint" type="fixed">
+    <link name="${robot_name}_camera_rgb_frame"/>
+    <joint name="${robot_name}_camera_rgb_optical_joint" type="fixed">
         <origin xyz="0 0 0" rpy="-1.57 0 -1.57"/>
-        <parent link="camera_rgb_frame"/>
-        <child link="camera_rgb_optical_frame"/>
+        <parent link="${robot_name}_camera_rgb_frame"/>
+        <child link="${robot_name}_camera_rgb_optical_frame"/>
     </joint>
-    <link name="camera_rgb_optical_frame"/>
-    <joint name="camera_depth_joint" type="fixed">
+    <link name="${robot_name}_camera_rgb_optical_frame"/>
+    <joint name="${robot_name}_camera_depth_joint" type="fixed">
         <origin xyz="${r200_cam_rgb_px} ${r200_cam_rgb_py + r200_cam_depth_offset} ${r200_cam_rgb_pz}" rpy="0 0 0"/>
-        <parent link="camera_link"/>
-        <child link="camera_depth_frame"/>
+        <parent link="${robot_name}_camera_link"/>
+        <child link="${robot_name}_camera_depth_frame"/>
     </joint>
-    <link name="camera_depth_frame"/>
-    <joint name="camera_depth_optical_joint" type="fixed">
+    <link name="${robot_name}_camera_depth_frame"/>
+    <joint name="${robot_name}_camera_depth_optical_joint" type="fixed">
         <origin xyz="0 0 0" rpy="-1.57 0 -1.57"/>
-        <parent link="camera_depth_frame"/>
-        <child link="camera_depth_optical_frame"/>
+        <parent link="${robot_name}_camera_depth_frame"/>
+        <child link="${robot_name}_camera_depth_optical_frame"/>
     </joint>
-    <link name="camera_depth_optical_frame"/>
+    <link name="${robot_name}_camera_depth_optical_frame"/>
 </robot>

File: urdf/wheel.urdf.xacro (robot description, xacro)
@@ -2,8 +2,10 @@
 <robot xmlns:xacro="http://www.ros.org/wiki/xacro" name="wheel">
   <!-- Properties -->
+  <xacro:arg name="robot_name" default="fella"/>
+  <xacro:property name="robot_name" value="$(arg robot_name)"/>
   <xacro:property name="wheel_separation" value="0.5708"/>
   <xacro:property name="wheel_radius" value="0.1651"/>
   <xacro:macro name="wheel" params="wheel_id x_pos y_pos">
-    <link name="${wheel_id}_wheel_link">
+    <link name="${robot_name}_${wheel_id}_wheel_link">
       <visual>
         <origin xyz="0 0 0" rpy="0 0 0"/>
@@ -28,7 +30,7 @@
     </link>
     <!-- Add joint to main body -->
-    <joint name="${wheel_id}_wheel_joint" type="revolute">
-      <parent link="base_link"/>
-      <child link="${wheel_id}_wheel_link" />
+    <joint name="${robot_name}_${wheel_id}_wheel_joint" type="revolute">
+      <parent link="${robot_name}_base_link"/>
+      <child link="${robot_name}_${wheel_id}_wheel_link" />
       <origin xyz="${x_pos} ${y_pos} 0.03282" rpy="0 0 0"/>
       <limit lower="-1e+16" upper="1e+16" effort="1e+16" velocity="1e+16"/>

Commit message: back wheel added to main

File: urdf/fella.urdf.xacro (robot description, xacro)
@@ -23,5 +23,5 @@
         </collision>
         <inertial>
-            <origin xyz="0 0 0.03282" rpy="0 0 0"/>
+            <origin xyz="-0.1 0 0.03282" rpy="0 0 0"/>
             <mass value="20.0"/>
             <inertia
@@ -37,4 +37,6 @@
     <xacro:wheel wheel_id="left" y_pos="0.42" x_pos="0.0"/>
     <xacro:wheel wheel_id="right" y_pos="-0.42" x_pos="0.0"/>
+    <!-- back wheels -->
+    <xacro:wheel wheel_id="back" y_pos="0.0" x_pos="-0.28"/>
     <joint name="imu_joint" type="fixed">
         <parent link="base_link"/>
